File: Le Chisoffre.kicad_pcb (KiCad board)
At the start: 2 copper layers, 236.5 x 103.2 mm, 129 parts, among them IC1 W25Q16JVUXIQ, J1 USB_C_Receptacle_USB2.0, J2 VIK Cirque Connector, SW1 boot, SW2 RotaryEncoder_Switch, U1 USBLC6-2SC6, U2 XC6206PxxxMR-Regulator_Linear, U3 RP2040, U4 XC6206P202MR, U5 PMW3360DM-T2QU_1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

Commit message: wip update
Parts:
- added H1: MountingHole, MountingHole:MountingHole_2.2mm_M2_DIN965_Pad, F.Cu at (134.8, 73.3)
- added H2: MountingHole, MountingHole:MountingHole_2.2mm_M2_DIN965_Pad, F.Cu at (166.9, 73.3)
- added H3: MountingHole, MountingHole:MountingHole_2.2mm_M2_DIN965_Pad, F.Cu at (134.9, 105.3)
- added H4: MountingHole, MountingHole:MountingHole_2.2mm_M2_DIN965_Pad, F.Cu at (166.9, 105.3)
- moved R2 4.76 mm to (158.0, 42.1)
- moved R5 4.76 mm to (143.7, 42.1)
- moved SW1 4.76 mm to (163.5, 42.1)
- moved SWR1 4.76 mm to (138.1, 42.1)
- moved C7 3.39 mm to (144.5, 50.1)
- moved C16 3.39 mm to (144.5, 45.1)
- moved C17 3.39 mm to (144.5, 51.1)
- moved U2 3.39 mm to (144.5, 47.6)
- moved R10 0.82 mm to (142.9, 83.5), turned to 180 degrees
- moved SWD1 0.79 mm to (144.5, 70.0)
Connections:
- U3 pad 11: /GPIO8 -> COL10
- U3 pad 12: /GPIO9 -> rot_a
- U3 pad 13: /GPIO10 -> rot_b
- U3 pad 2: /GPIO0 -> COL9
- U3 pad 27: /GPIO16 -> SDA
- U3 pad 28: /GPIO17 -> SCL
- U3 pad 29: /GPIO18 -> SCK
- U3 pad 3: /GPIO1 -> COL8
- U3 pad 30: /GPIO19 -> MOSI
- U3 pad 31: /GPIO20 -> MISO
- U3 pad 32: /GPIO21 -> CS
- U3 pad 35: /GPIO23 -> ROW3
- U3 pad 36: /GPIO24 -> ROW0
- U3 pad 37: /GPIO25 -> COL4
- U3 pad 38: /GPIO26 -> COL3
- U3 pad 39: /GPIO27 -> COL2
- U3 pad 4: /GPIO2 -> COL7
- U3 pad 40: /GPIO28 -> COL1
- U3 pad 41: /GPIO29 -> COL0
- U3 pad 5: /GPIO3 -> COL6
- U3 pad 6: /GPIO4 -> COL5
- U3 pad 7: /GPIO5 -> ROW1
- U3 pad 8: /GPIO6 -> ROW2
Routing:
- net MOSI: track 51.8 -> 83.6 mm, vias 1 -> 3
- net ROW3: track 326.9 -> 357.7 mm
- net CS: track 23.9 -> 52.8 mm, vias 0 -> 2
- net MISO: track 26.9 -> 55.5 mm, vias 0 -> 2
- net ROW2: track 352.4 -> 378.1 mm
- net ROW1: track 360.8 -> 383.7 mm
- net SCK: track 29.3 -> 51.9 mm, vias 0 -> 2
- net SDA: track 5.46 -> 28.0 mm, vias 0 -> 2
- net GND: track 82.6 -> 105.2 mm
- net COL0: track 131.0 -> 151.6 mm
- net COL1: track 136.9 -> 156.7 mm
- net COL6: track 92.4 -> 112.0 mm
- net COL8: track 133.2 -> 152.6 mm
- net COL7: track 116.3 -> 135.6 mm
- net COL9: track 125.4 -> 144.6 mm
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Other:
- outline, holes or cut-outs redrawn
- board text added: "2"
- board text added: "boot"
- board text added: "clk"
- board text added: "debug"
- board text added: "dio"
- board text added: "encoder"
- board text added: "reset"
- board text added: "sensor"

Commit message: update
first full version done
Parts:
- H1, H2, H3, H4: footprint MountingHole:MountingHole_2.2mm_M2_DIN965_Pad -> MountingHole:MountingHole_3.2mm_M3
- moved D37 1.03 mm to (118.7, 120.1)
- moved C15 0.79 mm to (156.4, 53.7)
- moved C21 0.20 mm to (161.9, 83.7)
Routing:
- net +3V3: track 138.3 -> 148.9 mm, vias 9 -> 10
- net GND: track 105.2 -> 113.8 mm
- net ROW0: track 351.0 -> 349.4 mm
- net MISO: track 55.5 -> 54.1 mm
- net MOSI: track 83.6 -> 84.7 mm
- net rot_b: track 35.0 -> 36.0 mm
- net Net-(D37-A): track 5.53 -> 6.53 mm
- net ROW1: track 383.7 -> 382.9 mm
- net COL10: track 73.2 -> 73.8 mm
Other:
- board text added: "SENSOR"
- board text removed: "sensor"

Commit message: clean up
Parts:
- removed MX41: MX_SW_solder, PCM_marbastlib-mx:SW_MX_1u
