File: Le Chisoffre.kicad_sch (KiCad schematic)
At the start: 118 parts, among them IC1 W25Q16JVUXIQ, J1 USB_C_Receptacle_USB2.0, SW1 boot, SW2 RotaryEncoder_Switch, U1 USBLC6-2SC6, U2 XC6206PxxxMR-Regulator_Linear, U3 RP2040, Y1 12MHz

Commit message: wip update
Connections:
- net GPIO0 is gone; now on net COL9: U3.2 (GPIO0)
- net GPIO1 is gone; now on net COL8: U3.3 (GPIO1)
- net GPIO10 is gone; now on net rot_b: U3.13 (GPIO10)
- net GPIO2 is gone; now on net COL7: U3.4 (GPIO2)
- net GPIO23 is gone; now on net ROW3: U3.35 (GPIO23)
- net GPIO24 is gone; now on net ROW0: U3.36 (GPIO24)
- net GPIO25 is gone; now on net COL4: U3.37 (GPIO25)
- net GPIO26 is gone; now on net COL3: U3.38 (GPIO26/ADC0)
- net GPIO27 is gone; now on net COL2: U3.39 (GPIO27/ADC1)
- net GPIO28 is gone; now on net COL1: U3.40 (GPIO28/ADC2)
- net GPIO29 is gone; now on net COL0: U3.41 (GPIO29/ADC3)
- net GPIO3 is gone; now on net COL6: U3.5 (GPIO3)
- net GPIO4 is gone; now on net COL5: U3.6 (GPIO4)
- net GPIO5 is gone; now on net ROW1: U3.7 (GPIO5)
- net GPIO6 is gone; now on net ROW2: U3.8 (GPIO6)
- net GPIO8 is gone; now on net COL10: U3.11 (GPIO8)
- net GPIO9 is gone; now on net rot_a: U3.12 (GPIO9)
- net GPIO16 renamed SDA
- net GPIO17 renamed SCL
- net GPIO18 renamed SCK
- net GPIO19 renamed MOSI
- net GPIO20 renamed MISO
- net GPIO21 renamed CS
- no-connect marks 3 -> 10

Commit message: backup
Parts:
- removed MX41: MX_SW_solder, PCM_marbastlib-mx:SW_MX_1u, symbol PCM_marbastlib-mx:MX_SW_solder
Changed lines of the file:
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@@
-	)
-	(symbol
-		(lib_id "PCM_marbastlib-mx:MX_SW_solder")
-		(at 209.55 73.66 0)
-		(unit 1)
-		(exclude_from_sim no)
-		(in_bom yes)
-		(on_board yes)
-		(dnp no)
-		(property "Reference" "MX41"
-			(at 209.55 69.596 0)
-			(effects
-				(font
-					(size 1.27 1.27)
-				)
-			)
-		)
-		(property "Value" "MX_SW_solder"
-			(at 209.55 68.58 0)
-			(effects
-				(font
-					(size 1.27 1.27)
-				)
-				(hide yes)
-			)
-		)
-		(property "Footprint" "PCM_marbastlib-mx:SW_MX_1u"
-			(at 209.55 73.66 0)
-			(effects
-				(font
-					(size 1.27 1.27)
-				)
-				(hide yes)
-			)
-		)
-		(property "Datasheet" "~"
-			(at 209.55 73.66 0)
-			(effects
-				(font
-					(size 1.27 1.27)
-				)
-				(hide yes)
-			)
-		)
-		(property "Description" "Push button switch, normally open, two pins, 45° tilted"
-			(at 209.55 73.66 0)
-			(effects
-				(font
-					(size 1.27 1.27)
-				)
-				(hide yes)
-			)
-		)
-		(pin "1"
-		)
-		(pin "2"
-		)
-		(instances
-			(project ""
-				(path "/1b359c20-7ce0-4923-93db-3e704c7c3bfa"
-					(reference "MX41")
-					(unit 1)
-				)
-			)
-		)
 	)
 	(symbol
