File: Project/Le Chisoffre.kicad_pcb (KiCad board)
At the start: 2 copper layers, 236.5 x 103.2 mm, 132 parts, among them IC1 W25Q16JVUXIQ, J1 USB_C_Receptacle_USB2.0, J2 VIK Cirque Connector, SW1 boot, SW2 RotaryEncoder_Switch, U1 USBLC6-2SC6, U2 XC6206PxxxMR-Regulator_Linear, U3 RP2040, U4 XC6206P202MR, U5 PMW3360DM-T2QU_1, Y1 12MHz

Commit message: finalised
Parts:
- added G***: LOGO, LOGO, B.Cu at (146.0, 117.4)
Routing:
- net ROW3: track 357.7 -> 356.6 mm
Other:
- board text added: "Calvin0563"
- board text added: "JLCJLCJLCJLC"
- board text added: "Le Chisoffre"
- board text added: "layout by haha"
- board text added: "pcb by"

Commit message: pcb finalized, cleanup necessary
Parts:
- removed G***: LOGO, LOGO
- removed S1, S2: MX_stab, PCM_marbastlib-mx:STAB_MX_P_ISO
- C1: value 100n -> 100nF
- MX1, MX10, MX11, MX12, MX13, MX14, MX15, MX16, MX17, MX18, MX19, MX2, MX20, MX21, MX22, MX23, MX24, MX25, MX26, MX27, MX28, MX29, MX3, MX30, MX33, MX34, MX4, MX5, MX6, MX7, MX8, MX9: footprint PCM_marbastlib-mx:SW_MX_1u -> PCM_marbastlib-mx:SW_MX_HS_S_CPG151101S11_1u
- MX31, MX32, MX35, MX36, MX37, MX40: footprint PCM_marbastlib-mx:SW_MX_1.25u -> PCM_marbastlib-mx:SW_MX_HS_S_CPG151101S11_1u
- MX38, MX39: footprint PCM_marbastlib-mx:SW_MX_1.5u -> PCM_marbastlib-mx:SW_MX_HS_S_CPG151101S11_1u
- moved D37 2.86 mm to (116.1, 121.1)
- moved D39 2.25 mm to (167.4, 122.2)
- moved MX1 0.70 mm to (50.7, 49.1)
- moved MX11 0.70 mm to (47.4, 67.8)
- moved MX12 0.70 mm to (67.0, 66.5)
- moved MX13 0.70 mm to (86.9, 63.2)
- moved MX14 0.70 mm to (104.5, 73.1)
- moved MX15 0.70 mm to (123.2, 76.4)
- moved MX2 0.70 mm to (70.3, 47.7)
- moved MX21 0.70 mm to (44.1, 86.6)
- moved MX22 0.70 mm to (63.7, 85.2)
- moved MX24 0.70 mm to (101.2, 91.8)
- moved MX25 0.70 mm to (119.9, 95.1)
- moved MX3 0.70 mm to (90.2, 44.4)
- moved MX31 0.70 mm to (79.8, 103.1)
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Routing:
- net ROW0: track 349.4 -> 243.8 mm
- net ROW2: track 378.5 -> 292.1 mm
- net ROW1: track 382.9 -> 304.7 mm
- net COL5: track 99.0 -> 108.0 mm
- net Net-(D38-A): track 22.6 -> 30.5 mm
- net Net-(D39-A): track 18.1 -> 25.5 mm
- net COL2: track 146.5 -> 152.9 mm
- net ROW3: track 356.6 -> 362.6 mm
- net COL6: track 112.0 -> 107.6 mm
- net COL3: track 118.7 -> 122.7 mm
- net COL0: track 151.6 -> 155.5 mm
- net Net-(D37-A): track 6.53 -> 10.2 mm
- net COL1: track 156.7 -> 160.4 mm
- net COL4: track 116.8 -> 120.0 mm
- net COL7: track 135.6 -> 137.5 mm
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Other:
- board size 236.5 x 103.2 mm -> 235.9 x 103.3 mm
- board text removed: "Calvin0563"
- board text removed: "JLCJLCJLCJLC"
- board text removed: "Le Chisoffre"
- board text removed: "layout by haha"
- board text removed: "pcb by"
